Commit message: moved the lasers to the center of the drone formated

File: urdf/quadrotor_with_two_hokuyo_utm30lx.urdf.xacro (robot description, xacro)
@@ -1,23 +1,28 @@
 <?xml version="1.0"?>
 <robot name="quadrotor" xmlns:xacro="http://www.ros.org/wiki/xacro">
-    <xacro:property name="M_PI" value="3.1415926535897931" />
-    <!-- Included URDF Files -->
-    <xacro:include filename="$(find hector_quadrotor_description)/urdf/quadrotor_base.urdf.xacro" />
-    <!-- Instantiate quadrotor_base_macro once (has no parameters atm) -->
-    <xacro:quadrotor_base_macro />
-    <!-- Hokuyo UTM-30LX mounted upside down below the quadrotor body -->
-    <xacro:include filename="$(find hector_sensors_description)/urdf/hokuyo_utm30lx.urdf.xacro" />
-    <xacro:hokuyo_utm30lx name="laser_up" parent="base_link" ros_topic="scan_up" update_rate="60" ray_count="181" min_angle="-90" max_angle="90">
-      <origin xyz="0.06 0.0 0.05" rpy="0 ${-M_PI/4} 0"/>
-    </xacro:hokuyo_utm30lx>
-    <!-- Hokuyo UTM-30LX mounted upside down below the quadrotor body
-    <xacro:include filename="$(find hector_sensors_description)/urdf/hokuyo_utm30lx.urdf.xacro" />
-    <xacro:hokuyo_utm30lx name="laser_up2" parent="base_link" ros_topic="scan_up2" update_rate="40" ray_count="1081" min_angle="-135" max_angle="135">
-      <origin xyz="0.06 0.0 0.05" rpy="0 ${-M_PI/6} 0"/>
+  <xacro:property name="M_PI" value="3.1415926535897931" />
+  <!-- Included URDF Files -->
+  <xacro:include filename="$(find hector_quadrotor_description)/urdf/quadrotor_base.urdf.xacro" />
+  <!-- Instantiate quadrotor_base_macro once (has no parameters atm) -->
+  <xacro:quadrotor_base_macro />
+  <!-- Hokuyo UTM-30LX mounted upside down below the quadrotor body -->
+  <xacro:include filename="$(find hector_sensors_description)/urdf/hokuyo_utm30lx.urdf.xacro" />
+  <xacro:hokuyo_utm30lx name="laser_up" parent="base_link" ros_topic="scan_up" update_rate="60"
+    ray_count="181" min_angle="-90" max_angle="90">
+    <origin xyz="0.00 0.0 0.05" rpy="0 ${-M_PI/4} 0" />
+  </xacro:hokuyo_utm30lx>
+  <!-- Hokuyo UTM-30LX mounted upside down below the quadrotor body
+    <xacro:include
+  filename="$(find hector_sensors_description)/urdf/hokuyo_utm30lx.urdf.xacro" />
+  <xacro:hokuyo_utm30lx name="laser_up2" parent="base_link" ros_topic="scan_up2" update_rate="40"
+  ray_count="1081" min_angle="-135" max_angle="135">
+      <origin xyz="0.06 0.0 0.05" rpy="0
+  ${-M_PI/6} 0"/>
     </xacro:hokuyo_utm30lx>-->
-    <!-- Hokuyo UTM-30LX mounted upside down below the quadrotor body -->
-    <xacro:include filename="$(find hector_sensors_description)/urdf/hokuyo_utm30lx.urdf.xacro" />
-    <xacro:hokuyo_utm30lx name="laser_down" parent="base_link" ros_topic="scan_down" update_rate="60" ray_count="181" min_angle="-90" max_angle="90">
-      <origin xyz="0.06 0.0 -0.05" rpy="${M_PI} ${M_PI/4} 0"/>
-    </xacro:hokuyo_utm30lx>
+  <!-- Hokuyo UTM-30LX mounted upside down below the quadrotor body -->
+  <xacro:include filename="$(find hector_sensors_description)/urdf/hokuyo_utm30lx.urdf.xacro" />
+  <xacro:hokuyo_utm30lx name="laser_down" parent="base_link" ros_topic="scan_down" update_rate="60"
+    ray_count="181" min_angle="-90" max_angle="90">
+    <origin xyz="0.00 0.0 -0.05" rpy="${M_PI} ${M_PI/4} 0" />
+  </xacro:hokuyo_utm30lx>
 </robot>
